File: cudrone-board-mk-2.brd (EAGLE design)
At the start: 100 x 70 mm, 60 parts, among them Q1 BSS138, U1 EDISON_CONNECTOR_FULLMOUNTING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, U2 FTS31XS-U, U4 TPS62065, U5 USD-SOCKETNEW, U6 TXB0108, U8 PCA9306, U9 MIC5205

Commit message: Added connectors to schematic
Parts:
- added ESC, RECIVER: 3X8, Drone_Connectors:3X8
- added SERVOS: 3X4, Drone_Connectors:3X4
Connections:
- new net AUX_0: RECIVER.S4
- new net AUX_1: RECIVER.S3
- new net AUX_2: RECIVER.S2
- new net AUX_3: RECIVER.S1
- new net M1: ESC.S8
- new net M2: ESC.S7
- new net M3: ESC.S6
- new net M4: ESC.S5
- new net M5: ESC.S4
- new net M6: ESC.S3
- new net M7: ESC.S2
- new net M8: ESC.S1
- new net PITCH: RECIVER.S8
- new net ROLL: RECIVER.S7
- new net THROTTLE: RECIVER.S5
- new net YAW: RECIVER.S6
- net 5V: now also ESC.V1, ESC.V2, ESC.V3, ESC.V4, ESC.V5, ESC.V6, ESC.V7, ESC.V8, RECIVER.V1, RECIVER.V2, RECIVER.V3, RECIVER.V4, RECIVER.V5, RECIVER.V6, RECIVER.V7, RECIVER.V8, SERVOS.V1, SERVOS.V2, SERVOS.V3, SERVOS.V4
- net GND: now also ESC.G1, ESC.G2, ESC.G3, ESC.G4, ESC.G5, ESC.G6, ESC.G7, ESC.G8, RECIVER.G1, RECIVER.G2, RECIVER.G3, RECIVER.G4, RECIVER.G5, RECIVER.G6, RECIVER.G7, RECIVER.G8, SERVOS.G1, SERVOS.G2, SERVOS.G3, SERVOS.G4
- net GP12_PWM0: now also SERVOS.S4
- net GP13_PWM1: now also SERVOS.S3
- net GP182_PWM2: now also SERVOS.S2
- net GP183_PWM3: now also SERVOS.S1
Changed lines of the file:
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@@
 <layer number="113" name="IDFDebug" color="7" fill="1" visible="yes" active="yes"/>
 <layer number="114" name="Badge_Outline" color="11" fill="1" visible="no" active="no"/>
+<layer number="115" name="ReferenceISLANDS" color="7" fill="1" visible="yes" active="yes"/>
 <layer number="116" name="Patch_BOT" color="9" fill="4" visible="yes" active="yes"/>
 <layer number="118" name="Rect_Pads" color="7" fill="1" visible="yes" active="yes"/>
@@
 <attribute name="PROD_ID" value="RES-08272" x="-96" y="-218" size="1.778" layer="27" display="off"/>
 </element>
+<element name="SERVOS" library="Drone_Connectors" package="3X4" value="3X4" x="-69" y="-219"/>
+<element name="RECIVER" library="Drone_Connectors" package="3X8" value="3X8" x="-63" y="-227"/>
+<element name="ESC" library="Drone_Connectors" package="3X8" value="3X8" x="-63" y="-235"/>
 </elements>
 <signals>
@@
 <contactref element="C14" pad="2"/>
 <contactref element="U9" pad="2"/>
+<contactref element="SERVOS" pad="G2"/>
+<contactref element="SERVOS" pad="G3"/>
+<contactref element="SERVOS" pad="G1"/>
+<contactref element="SERVOS" pad="G4"/>
+<contactref element="RECIVER" pad="G7"/>
+<contactref element="RECIVER" pad="G6"/>
+<contactref element="RECIVER" pad="G8"/>
+<contactref element="RECIVER" pad="G3"/>
+<contactref element="RECIVER" pad="G2"/>
+<contactref element="RECIVER" pad="G4"/>
+<contactref element="RECIVER" pad="G5"/>
+<contactref element="RECIVER" pad="G1"/>
+<contactref element="ESC" pad="G7"/>
+<contactref element="ESC" pad="G6"/>
+<contactref element="ESC" pad="G8"/>
+<contactref element="ESC" pad="G3"/>
+<contactref element="ESC" pad="G2"/>
+<contactref element="ESC" pad="G4"/>
+<contactref element="ESC" pad="G5"/>
+<contactref element="ESC" pad="G1"/>
 <wire x1="-67.15" y1="-178" x2="-72.8" y2="-178.1" width="0" layer="19" extent="1-1"/>
 <wire x1="-63.15" y1="-178" x2="-67.15" y2="-178" width="0" layer="19" extent="1-1"/>
@@
 <wire x1="-69.15" y1="-210" x2="-67.6" y2="-206" width="0" layer="19" extent="1-1"/>
 <wire x1="-73.15" y1="-210" x2="-69.15" y2="-210" width="0" layer="19" extent="1-1"/>
+<wire x1="-72.81" y1="-221.54" x2="-73.15" y2="-210" width="0" layer="19" extent="1-1"/>
+<wire x1="-70.27" y1="-221.54" x2="-72.81" y2="-221.54" width="0" layer="19" extent="1-1"/>
+<wire x1="-67.73" y1="-221.54" x2="-70.27" y2="-221.54" width="0" layer="19" extent="1-1"/>
+<wire x1="-65.19" y1="-221.54" x2="-67.73" y2="-221.54" width="0" layer="19" extent="1-1"/>
+<wire x1="-71.89" y1="-229.54" x2="-72.81" y2="-221.54" width="0" layer="19" extent="1-1"/>
+<wire x1="-69.35" y1="-229.54" x2="-71.89" y2="-229.54" width="0" layer="19" extent="1-1"/>
+<wire x1="-66.81" y1="-229.54" x2="-69.35" y2="-229.54" width="0" layer="19" extent="1-1"/>
+<wire x1="-64.27" y1="-229.54" x2="-66.81" y2="-229.54" width="0" layer="19" extent="1-1"/>
+<wire x1="-61.73" y1="-229.54" x2="-64.27" y2="-229.54" width="0" layer="19" extent="1-1"/>
+<wire x1="-59.19" y1="-229.54" x2="-61.73" y2="-229.54" width="0" layer="19" extent="1-1"/>
+<wire x1="-56.65" y1="-229.54" x2="-59.19" y2="-229.54" width="0" layer="19" extent="1-1"/>
+<wire x1="-54.11" y1="-229.54" x2="-56.65" y2="-229.54" width="0" layer="19" extent="1-1"/>
+<wire x1="-71.89" y1="-237.54" x2="-71.89" y2="-229.54" width="0" layer="19" extent="1-1"/>
+<wire x1="-69.35" y1="-237.54" x2="-71.89" y2="-237.54" width="0" layer="19" extent="1-1"/>
+<wire x1="-66.81" y1="-237.54" x2="-69.35" y2="-237.54" width="0" layer="19" extent="1-1"/>
+<wire x1="-64.27" y1="-237.54" x2="-66.81" y2="-237.54" width="0" layer="19" extent="1-1"/>
+<wire x1="-61.73" y1="-237.54" x2="-64.27" y2="-237.54" width="0" layer="19" extent="1-1"/>
+<wire x1="-59.19" y1="-237.54" x2="-61.73" y2="-237.54" width="0" layer="19" extent="1-1"/>
+<wire x1="-56.65" y1="-237.54" x2="-59.19" y2="-237.54" width="0" layer="19" extent="1-1"/>
+<wire x1="-54.11" y1="-237.54" x2="-56.65" y2="-237.54" width="0" layer="19" extent="1-1"/>
 <wire x1="-65.44" y1="-164.1" x2="-67.15" y2="-178" width="0" layer="19" extent="1-1"/>
 <wire x1="-62.45" y1="-161.45" x2="-65.44" y2="-164.1" width="0" layer="19" extent="1-1"/>
@@
 <signal name="GP183_PWM3">
 <contactref element="U1" pad="39"/>
+<contactref element="SERVOS" pad="S1"/>
+<wire x1="-72.81" y1="-216.46" x2="43.57" y2="47.02" width="0" layer="19" extent="1-1"/>
 </signal>
 <signal name="GP182_PWM2">
 <contactref element="U1" pad="37"/>
+<contactref element="SERVOS" pad="S2"/>
+<wire x1="-70.27" y1="-216.46" x2="43.97" y2="47.02" width="0" layer="19" extent="1-1"/>
 </signal>
 <signal name="GP13_PWM1">
 <contactref element="U1" pad="33"/>
+<contactref element="SERVOS" pad="S3"/>
+<wire x1="-67.73" y1="-216.46" x2="44.77" y2="47.02" width="0" layer="19" extent="1-1"/>
 </signal>
 <signal name="GP12_PWM0">
 <contactref element="U1" pad="35"/>
+<contactref element="SERVOS" pad="S4"/>
+<wire x1="-65.19" y1="-216.46" x2="44.37" y2="47.02" width="0" layer="19" extent="1-1"/>
 </signal>
 <signal name="GP14">
@@
 <contactref element="D4" pad="C"/>
 <contactref element="U$3" pad="1"/>
+<contactref element="SERVOS" pad="V1"/>
+<contactref element="SERVOS" pad="V3"/>
+<contactref element="SERVOS" pad="V2"/>
+<contactref element="SERVOS" pad="V4"/>
+<contactref element="RECIVER" pad="V7"/>
+<contactref element="RECIVER" pad="V6"/>
+<contactref element="RECIVER" pad="V3"/>
+<contactref element="RECIVER" pad="V1"/>
+<contactref element="RECIVER" pad="V4"/>
+<contactref element="RECIVER" pad="V8"/>
+<contactref element="RECIVER" pad="V5"/>
+<contactref element="RECIVER" pad="V2"/>
+<contactref element="ESC" pad="V7"/>
+<contactref element="ESC" pad="V6"/>
+<contactref element="ESC" pad="V3"/>
+<contactref element="ESC" pad="V1"/>
+<contactref element="ESC" pad="V4"/>
+<contactref element="ESC" pad="V8"/>
+<contactref element="ESC" pad="V5"/>
+<contactref element="ESC" pad="V2"/>
 <wire x1="-65.95" y1="-138.3751" x2="-70.85" y2="-148" width="0" layer="19" extent="1-1"/>
 <wire x1="-69.15" y1="-132" x2="-65.95" y2="-138.3751" width="0" layer="19" extent="1-1"/>
@@
 <wire x1="-75.75" y1="-93.05" x2="-75.25" y2="-93.05" width="0" layer="19" extent="1-1"/>
 <wire x1="-74.9" y1="-87" x2="-75.25" y2="-93.05" width="0" layer="19" extent="1-1"/>
+<wire x1="-70.27" y1="-219" x2="-70.85" y2="-148" width="0" layer="19" extent="1-1"/>
+<wire x1="-72.81" y1="-219" x2="-70.27" y2="-219" width="0" layer="19" extent="1-1"/>
+<wire x1="-67.73" y1="-219" x2="-70.27" y2="-219" width="0" layer="19" extent="1-1"/>
+<wire x1="-65.19" y1="-219" x2="-67.73" y2="-219" width="0" layer="19" extent="1-1"/>
+<wire x1="-71.89" y1="-227" x2="-72.81" y2="-219" width="0" layer="19" extent="1-1"/>
+<wire x1="-69.35" y1="-227" x2="-71.89" y2="-227" width="0" layer="19" extent="1-1"/>
+<wire x1="-66.81" y1="-227" x2="-69.35" y2="-227" width="0" layer="19" extent="1-1"/>
+<wire x1="-64.27" y1="-227" x2="-66.81" y2="-227" width="0" layer="19" extent="1-1"/>
+<wire x1="-61.73" y1="-227" x2="-64.27" y2="-227" width="0" layer="19" extent="1-1"/>
+<wire x1="-59.19" y1="-227" x2="-61.73" y2="-227" width="0" layer="19" extent="1-1"/>
+<wire x1="-56.65" y1="-227" x2="-59.19" y2="-227" width="0" layer="19" extent="1-1"/>
+<wire x1="-54.11" y1="-227" x2="-56.65" y2="-227" width="0" layer="19" extent="1-1"/>
+<wire x1="-71.89" y1="-235" x2="-71.89" y2="-227" width="0" layer="19" extent="1-1"/>
+<wire x1="-69.35" y1="-235" x2="-71.89" y2="-235" width="0" layer="19" extent="1-1"/>
+<wire x1="-66.81" y1="-235" x2="-69.35" y2="-235" width="0" layer="19" extent="1-1"/>
+<wire x1="-64.27" y1="-235" x2="-66.81" y2="-235" width="0" layer="19" extent="1-1"/>
+<wire x1="-61.73" y1="-235" x2="-64.27" y2="-235" width="0" layer="19" extent="1-1"/>
+<wire x1="-59.19" y1="-235" x2="-61.73" y2="-235" width="0" layer="19" extent="1-1"/>
+<wire x1="-56.65" y1="-235" x2="-59.19" y2="-235" width="0" layer="19" extent="1-1"/>
+<wire x1="-54.11" y1="-235" x2="-56.65" y2="-235" width="0" layer="19" extent="1-1"/>
 </signal>
 <signal name="N$12">
@@
 <wire x1="-69.73" y1="-191.775" x2="-73.365" y2="-206" width="0" layer="19" extent="1-1"/>
 </signal>
+<signal name="PITCH">
+<contactref element="RECIVER" pad="S8"/>
+</signal>
+<signal name="ROLL">
+<contactref element="RECIVER" pad="S7"/>
+</signal>
+<signal name="YAW">
+<contactref element="RECIVER" pad="S6"/>
+</signal>
+<signal name="THROTTLE">
+<contactref element="RECIVER" pad="S5"/>
+</signal>
+<signal name="AUX_0">
+<contactref element="RECIVER" pad="S4"/>
+</signal>
+<signal name="AUX_1">
+<contactref element="RECIVER" pad="S3"/>
+</signal>
+<signal name="AUX_2">
+<contactref element="RECIVER" pad="S2"/>
+</signal>
+<signal name="AUX_3">
+<contactref element="RECIVER" pad="S1"/>
+</signal>
+<signal name="M1">
+<contactref element="ESC" pad="S8"/>
+</signal>
+<signal name="M2">
+<contactref element="ESC" pad="S7"/>
+</signal>
+<signal name="M3">
+<contactref element="ESC" pad="S6"/>
+</signal>
+<signal name="M4">
+<contactref element="ESC" pad="S5"/>
+</signal>
+<signal name="M5">
+<contactref element="ESC" pad="S4"/>
+</signal>
+<signal name="M6">
+<contactref element="ESC" pad="S3"/>
+</signal>
+<signal name="M7">
+<contactref element="ESC" pad="S2"/>
+</signal>
+<signal name="M8">
+<contactref element="ESC" pad="S1"/>
+</signal>
 </signals>

Commit message: Added new port for servos on the motors to be connected. Picked a dsp to be used to control the motors
Parts:
- added MOTOR_SERVO: 3X8, Drone_Connectors:3X8
- added U$4: DSPIC33EP512MC806-I/PT, DSPIC33EP512MC806:TQFP64_10X10MC
- renumbered SERVOS to GIMBAL_SERVOS
Connections:
- new net AVDD: U$4.19
- new net AVSS: U$4.20
- new net MS1: MOTOR_SERVO.S8
- new net MS2: MOTOR_SERVO.S7
- new net MS3: MOTOR_SERVO.S6
- new net MS4: MOTOR_SERVO.S5
- new net MS5: MOTOR_SERVO.S4
- new net MS6: MOTOR_SERVO.S3
- new net MS7: MOTOR_SERVO.S2
- new net MS8: MOTOR_SERVO.S1
- new net VCAP: U$4.56
- new net VDD: U$4.57
- new net VDD_2: U$4.10
- new net VDD_3: U$4.26
- new net VDD_4: U$4.38
- new net VSS: U$4.41
- new net VSS_2: U$4.9
- new net VSS_3: U$4.25
- net 5V: now also MOTOR_SERVO.V1, MOTOR_SERVO.V2, MOTOR_SERVO.V3, MOTOR_SERVO.V4, MOTOR_SERVO.V5, MOTOR_SERVO.V6, MOTOR_SERVO.V7, MOTOR_SERVO.V8
- net GND: now also MOTOR_SERVO.G1, MOTOR_SERVO.G2, MOTOR_SERVO.G3, MOTOR_SERVO.G4, MOTOR_SERVO.G5, MOTOR_SERVO.G6, MOTOR_SERVO.G7, MOTOR_SERVO.G8
Changed lines of the file:
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@@
 <?xml version="1.0" encoding="utf-8"?>
 <!DOCTYPE eagle SYSTEM "eagle.dtd">
-<eagle version="6.5.0">
+<eagle version="8.0.0">
 <drawing>
 <settings>
@@
 <layer number="59" name="tCarbon" color="7" fill="1" visible="no" active="no"/>
 <layer number="60" name="bCarbon" color="7" fill="1" visible="no" active="no"/>
-<layer number="90" name="Modules" color="5" fill="1" visible="yes" active="yes"/>
+<layer number="90" name="Modules" color="5" fill="1" visible="no" active="no"/>
 <layer number="91" name="Nets" color="2" fill="1" visible="no" active="no"/>
 <layer number="92" name="Busses" color="1" fill="1" visible="no" active="no"/>
@@
 <pass name="Default">
 <param name="RoutingGrid" value="50mil"/>
+<param name="AutoGrid" value="1"/>
+<param name="Efforts" value="0"/>
+<param name="TopRouterVariant" value="1"/>
 <param name="tpViaShape" value="round"/>
 <param name="PrefDir.1" value="|"/>
@@
 <attribute name="PROD_ID" value="RES-08272" x="-96" y="-218" size="1.778" layer="27" display="off"/>
 </element>
-<element name="SERVOS" library="Drone_Connectors" package="3X4" value="3X4" x="-69" y="-219"/>
+<element name="GIMBAL_SERVOS" library="Drone_Connectors" package="3X4" value="3X4" x="-69" y="-219"/>
 <element name="RECIVER" library="Drone_Connectors" package="3X8" value="3X8" x="-63" y="-227"/>
 <element name="ESC" library="Drone_Connectors" package="3X8" value="3X8" x="-63" y="-235"/>
+<element name="MOTOR_SERVO" library="Drone_Connectors" package="3X8" value="3X8" x="-63" y="-259"/>
+<element name="U$4" library="DSPIC33EP512MC806" package="TQFP64_10X10MC" value="DSPIC33EP512MC806-I/PT" x="-74" y="-278">
+<attribute name="VENDOR" value="MICROCHIP" x="-74" y="-278" size="1.778" layer="27" display="off"/>
+<attribute name="MANUFACTURER_PART_NUMBER" value="dspic33ep512mc806ipt" x="-74" y="-278" size="1.778" layer="27" display="off"/>
+</element>
 </elements>
 <signals>
@@
 <contactref element="C14" pad="2"/>
 <contactref element="U9" pad="2"/>
-<contactref element="SERVOS" pad="G2"/>
-<contactref element="SERVOS" pad="G3"/>
-<contactref element="SERVOS" pad="G1"/>
-<contactref element="SERVOS" pad="G4"/>
+<contactref element="GIMBAL_SERVOS" pad="G2"/>
+<contactref element="GIMBAL_SERVOS" pad="G3"/>
+<contactref element="GIMBAL_SERVOS" pad="G1"/>
+<contactref element="GIMBAL_SERVOS" pad="G4"/>
 <contactref element="RECIVER" pad="G7"/>
 <contactref element="RECIVER" pad="G6"/>
@@
 <contactref element="ESC" pad="G5"/>
 <contactref element="ESC" pad="G1"/>
+<contactref element="MOTOR_SERVO" pad="G3"/>
+<contactref element="MOTOR_SERVO" pad="G4"/>
+<contactref element="MOTOR_SERVO" pad="G1"/>
+<contactref element="MOTOR_SERVO" pad="G6"/>
+<contactref element="MOTOR_SERVO" pad="G7"/>
+<contactref element="MOTOR_SERVO" pad="G2"/>
+<contactref element="MOTOR_SERVO" pad="G5"/>
+<contactref element="MOTOR_SERVO" pad="G8"/>
 <wire x1="-67.15" y1="-178" x2="-72.8" y2="-178.1" width="0" layer="19" extent="1-1"/>
 <wire x1="-63.15" y1="-178" x2="-67.15" y2="-178" width="0" layer="19" extent="1-1"/>
@@
 <wire x1="-64.1" y1="-82" x2="-66.85" y2="-91" width="0" layer="19" extent="1-1"/>
 <wire x1="-66" y1="-67" x2="-64.1" y2="-82" width="0" layer="19" extent="1-1"/>
+<wire x1="-71.89" y1="-261.54" x2="-71.89" y2="-237.54" width="0" layer="19" extent="1-1"/>
+<wire x1="-69.35" y1="-261.54" x2="-71.89" y2="-261.54" width="0" layer="19" extent="1-1"/>
+<wire x1="-66.81" y1="-261.54" x2="-69.35" y2="-261.54" width="0" layer="19" extent="1-1"/>
+<wire x1="-64.27" y1="-261.54" x2="-66.81" y2="-261.54" width="0" layer="19" extent="1-1"/>
+<wire x1="-61.73" y1="-261.54" x2="-64.27" y2="-261.54" width="0" layer="19" extent="1-1"/>
+<wire x1="-59.19" y1="-261.54" x2="-61.73" y2="-261.54" width="0" layer="19" extent="1-1"/>
+<wire x1="-56.65" y1="-261.54" x2="-59.19" y2="-261.54" width="0" layer="19" extent="1-1"/>
+<wire x1="-54.11" y1="-261.54" x2="-56.65" y2="-261.54" width="0" layer="19" extent="1-1"/>
 <wire x1="48.37" y1="47.02" x2="-66" y2="-67" width="0" layer="19" extent="1-1"/>
 <wire x1="48.77" y1="47.02" x2="48.37" y2="47.02" width="0" layer="19" extent="1-1"/>
@@
 <signal name="GP183_PWM3">
 <contactref element="U1" pad="39"/>
-<contactref element="SERVOS" pad="S1"/>
+<contactref element="GIMBAL_SERVOS" pad="S1"/>
 <wire x1="-72.81" y1="-216.46" x2="43.57" y2="47.02" width="0" layer="19" extent="1-1"/>
 </signal>
 <signal name="GP182_PWM2">
 <contactref element="U1" pad="37"/>
-<contactref element="SERVOS" pad="S2"/>
+<contactref element="GIMBAL_SERVOS" pad="S2"/>
 <wire x1="-70.27" y1="-216.46" x2="43.97" y2="47.02" width="0" layer="19" extent="1-1"/>
 </signal>
 <signal name="GP13_PWM1">
 <contactref element="U1" pad="33"/>
-<contactref element="SERVOS" pad="S3"/>
+<contactref element="GIMBAL_SERVOS" pad="S3"/>
 <wire x1="-67.73" y1="-216.46" x2="44.77" y2="47.02" width="0" layer="19" extent="1-1"/>
 </signal>
 <signal name="GP12_PWM0">
 <contactref element="U1" pad="35"/>
-<contactref element="SERVOS" pad="S4"/>
+<contactref element="GIMBAL_SERVOS" pad="S4"/>
 <wire x1="-65.19" y1="-216.46" x2="44.37" y2="47.02" width="0" layer="19" extent="1-1"/>
 </signal>
@@
 <contactref element="D4" pad="C"/>
 <contactref element="U$3" pad="1"/>
-<contactref element="SERVOS" pad="V1"/>
-<contactref element="SERVOS" pad="V3"/>
-<contactref element="SERVOS" pad="V2"/>
-<contactref element="SERVOS" pad="V4"/>
+<contactref element="GIMBAL_SERVOS" pad="V1"/>
+<contactref element="GIMBAL_SERVOS" pad="V3"/>
+<contactref element="GIMBAL_SERVOS" pad="V2"/>
+<contactref element="GIMBAL_SERVOS" pad="V4"/>
 <contactref element="RECIVER" pad="V7"/>
 <contactref element="RECIVER" pad="V6"/>
@@
 <contactref element="ESC" pad="V5"/>
 <contactref element="ESC" pad="V2"/>
+<contactref element="MOTOR_SERVO" pad="V3"/>
+<contactref element="MOTOR_SERVO" pad="V7"/>
+<contactref element="MOTOR_SERVO" pad="V8"/>
+<contactref element="MOTOR_SERVO" pad="V4"/>
+<contactref element="MOTOR_SERVO" pad="V1"/>
+<contactref element="MOTOR_SERVO" pad="V5"/>
+<contactref element="MOTOR_SERVO" pad="V2"/>
+<contactref element="MOTOR_SERVO" pad="V6"/>
 <wire x1="-65.95" y1="-138.3751" x2="-70.85" y2="-148" width="0" layer="19" extent="1-1"/>
 <wire x1="-69.15" y1="-132" x2="-65.95" y2="-138.3751" width="0" layer="19" extent="1-1"/>
@@
 <wire x1="-56.65" y1="-235" x2="-59.19" y2="-235" width="0" layer="19" extent="1-1"/>
 <wire x1="-54.11" y1="-235" x2="-56.65" y2="-235" width="0" layer="19" extent="1-1"/>
+<wire x1="-71.89" y1="-259" x2="-71.89" y2="-235" width="0" layer="19" extent="1-1"/>
+<wire x1="-69.35" y1="-259" x2="-71.89" y2="-259" width="0" layer="19" extent="1-1"/>
+<wire x1="-66.81" y1="-259" x2="-69.35" y2="-259" width="0" layer="19" extent="1-1"/>
+<wire x1="-64.27" y1="-259" x2="-66.81" y2="-259" width="0" layer="19" extent="1-1"/>
+<wire x1="-61.73" y1="-259" x2="-64.27" y2="-259" width="0" layer="19" extent="1-1"/>
+<wire x1="-59.19" y1="-259" x2="-61.73" y2="-259" width="0" layer="19" extent="1-1"/>
+<wire x1="-56.65" y1="-259" x2="-59.19" y2="-259" width="0" layer="19" extent="1-1"/>
+<wire x1="-54.11" y1="-259" x2="-56.65" y2="-259" width="0" layer="19" extent="1-1"/>
 </signal>
 <signal name="N$12">
@@
 <contactref element="ESC" pad="S1"/>
 </signal>
+<signal name="MS1">
+<contactref element="MOTOR_SERVO" pad="S8"/>
+</signal>
+<signal name="MS2">
+<contactref element="MOTOR_SERVO" pad="S7"/>
+</signal>
+<signal name="MS3">
+<contactref element="MOTOR_SERVO" pad="S6"/>
+</signal>
+<signal name="MS4">
+<contactref element="MOTOR_SERVO" pad="S5"/>
+</signal>
+<signal name="MS5">
+<contactref element="MOTOR_SERVO" pad="S4"/>
+</signal>
+<signal name="MS6">
+<contactref element="MOTOR_SERVO" pad="S3"/>
+</signal>
+<signal name="MS7">
+<contactref element="MOTOR_SERVO" pad="S2"/>
+</signal>
+<signal name="MS8">
+<contactref element="MOTOR_SERVO" pad="S1"/>
+</signal>
+<signal name="VSS_2">
+<contactref element="U$4" pad="9"/>
+</signal>
+<signal name="VDD_2">
+<contactref element="U$4" pad="10"/>
+</signal>
+<signal name="AVDD">
+<contactref element="U$4" pad="19"/>
+</signal>
+<signal name="AVSS">
+<contactref element="U$4" pad="20"/>
+</signal>
+<signal name="VSS_3">
+<contactref element="U$4" pad="25"/>
+</signal>
+<signal name="VDD_3">
+<contactref element="U$4" pad="26"/>
+</signal>
+<signal name="VDD_4">
+<contactref element="U$4" pad="38"/>
+</signal>
+<signal name="VSS">
+<contactref element="U$4" pad="41"/>
+</signal>
+<signal name="VCAP">
+<contactref element="U$4" pad="56"/>
+</signal>
+<signal name="VDD">
+<contactref element="U$4" pad="57"/>
+</signal>
 </signals>

Commit message: Made their be a few less motor connectors so that everything fits on the dsp. Also added some reguator libraries
Parts:
- removed RECIVER: 3X8, Drone_Connectors:3X8
- removed S1: POWER, SparkFun-Electromechanical:TACTILE_SWITCH-SMD-RIGHT-ANGLE
- added GIMBAL_SERVOS1: 3X4, Drone_Connectors:3X4
- added POWER: CANSAT_SWITCH, SparkFun-Electromechanical:JS102011SAQN-SPDT
- D2: value YELLOW -> Yellow
- ESC, MOTOR_SERVO: value 3X8 -> 3X6; device Drone_Connectors:3X8 -> Drone_Connectors:3X6
- Q1: value BSS138 -> 200mA/50V
- R10, R11, R12, R15, R16, R17, R18, R19, R20, R3, R4, R5, R6, R7, R8, R9: device SparkFun-Resistors:0603-RES -> SparkFun-Resistors:0603-RES@1
- SJ4: device SparkFun-Passives:PAD-JUMPER-3-2OF3_NC_BY_TRACE_YES_SILK_FULL_BOX -> SparkFun-Passives:PAD-JUMPER-3-2OF3_NC_BY_TRACE_YES_SILK_LARGE
- moved ESC 86.1 mm to (-66.0, -321.0)
- moved MOTOR_SERVO 86.1 mm to (-66.0, -345.0)
- renumbered U$4 to MOTOR_CONTROLLER
Connections:
- removed net AUX_0: RECIVER.S4
- removed net AUX_1: RECIVER.S3
- removed net AUX_2: RECIVER.S2
- removed net AUX_3: RECIVER.S1
- removed net M7: ESC.S2
- removed net M8: ESC.S1
- removed net MS7: MOTOR_SERVO.S2
- removed net MS8: MOTOR_SERVO.S1
- net 3.3V: now also U5.VCC; no longer U5.4
- net 5V: now also GIMBAL_SERVOS1.V1, GIMBAL_SERVOS1.V2, GIMBAL_SERVOS1.V3, GIMBAL_SERVOS1.V4; no longer ESC.V7, ESC.V8, MOTOR_SERVO.V7, MOTOR_SERVO.V8, RECIVER.V1, RECIVER.V2, RECIVER.V3, RECIVER.V4, RECIVER.V5, RECIVER.V6, RECIVER.V7, RECIVER.V8
- net GND: now also GIMBAL_SERVOS1.G1, GIMBAL_SERVOS1.G2, GIMBAL_SERVOS1.G3, GIMBAL_SERVOS1.G4, POWER.P$1, U5.GND, U9.3; no longer ESC.G7, ESC.G8, MOTOR_SERVO.G7, MOTOR_SERVO.G8, RECIVER.G1, RECIVER.G2, RECIVER.G3, RECIVER.G4, RECIVER.G5, RECIVER.G6, RECIVER.G7, RECIVER.G8, S1.2, U5.6, U9.2
- net M1: now also ESC.S6; no longer ESC.S8
- net M2: now also ESC.S5; no longer ESC.S7
- net M3: now also ESC.S4; no longer ESC.S6
- net M4: now also ESC.S3; no longer ESC.S5
- net M5: now also ESC.S2; no longer ESC.S4
- net M6: now also ESC.S1; no longer ESC.S3
- net MS1: now also MOTOR_SERVO.S6; no longer MOTOR_SERVO.S8
- net MS2: now also MOTOR_SERVO.S5; no longer MOTOR_SERVO.S7
- net MS3: now also MOTOR_SERVO.S4; no longer MOTOR_SERVO.S6
- net MS4: now also MOTOR_SERVO.S3; no longer MOTOR_SERVO.S5
- net MS5: now also MOTOR_SERVO.S2; no longer MOTOR_SERVO.S4
- net MS6: now also MOTOR_SERVO.S1; no longer MOTOR_SERVO.S3
- net N$15: now also POWER.P$C; no longer S1.1
- net N$20: now also U5.RSV1; no longer U5.1
- net N$21: now also U5.CS; no longer U5.2
- net N$22: now also U5.DI; no longer U5.3
- net N$23: now also U5.DO; no longer U5.7
- net N$24: now also U5.RSV2; no longer U5.8
- net PITCH: now also GIMBAL_SERVOS1.S4; no longer RECIVER.S8
- net ROLL: now also GIMBAL_SERVOS1.S3; no longer RECIVER.S7
- net SCK: now also U5.SCLK; no longer U5.5
- net THROTTLE: now also GIMBAL_SERVOS1.S1; no longer RECIVER.S5
- net VSYS: now also U9.2; no longer U9.3
- net YAW: now also GIMBAL_SERVOS1.S2; no longer RECIVER.S6
