File: cudrone-board-mk-2.brd (EAGLE design)
At the start: 100 x 70 mm, 65 parts, among them Q1 200mA/50V, U1 EDISON_CONNECTOR_FULLMOUNTING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, U2 FTS31XS-U, U4 TPS62065, U5 USD-SOCKETNEW, U6 TXB0108, U8 PCA9306, U9 MIC5205

Commit message: Added logic level shifters to servos and changed how power input works
Parts:
- removed Q1: 200mA/50V, SparkFun-DiscreteSemi:SOT23-3
- added BSS138_1, BSS138_2, BSS138_3, BSS138_7: PMV22EN, eagle-library-edeca.net-v5:SOT23
- added C15, C16: 47pF, SparkFun-Capacitors:0603-CAP
- added D5: RED, SparkFun-LED:LED-0603
- added D6: Yellow, SparkFun-LED:LED-0603
- added R21: 10K, SparkFun-Resistors:0603-RES@1
- added R22: 200k, SparkFun-Resistors:0603-RES@1
- added R23, R24: DNP, SparkFun-Resistors:0603-RES@1
- added R25, R26: 27, SparkFun-Resistors:0603
- added R27, R28: 1K, SparkFun-Resistors:0603-RES@1
- added R29, R30: 100, SparkFun-Resistors:0603-RES@1
- added R31, R32, R33, R34, R35, R36, R37, R38, R39, R40, R41, R42: (no value), SparkFun-Passives:0603-RES
- added R43, R44, R45, R46, R47, R48, R49, R50: 10k, SparkFun-Resistors:0805
- added RESET: SWITCH-MOMENTARY-2PTH, SparkFun-Electromechanical:TACTILE-PTH
- added SJ5: JUMPER-PAD-2-NC_BY_TRACE, SparkFun-Passives:PAD-JUMPER-2-NC_BY_TRACE_YES_SILK
- added U10: A2235-H, A2235-H:XCVR_A2235-H
- added U11: FTS31XS-U, SparkFun-DigitalIC:SSOP20_L
- C13, C14: value 10uF -> 0.1uF; device SparkFun-Capacitors:1206 -> SparkFun-Capacitors:0603-CAP
- JP2: value (none) -> USB_MICROB; device SparkFun-Connectors:1X04_SMD_RA_FEMALE -> SparkFun-Connectors:USB-B-MICRO-SMD_V03
- R14: value 120k -> 150k
- R15: value 1K -> 10K
- SJ4: value Power Select -> JUMPER-PAD-2-NC_BY_TRACE; device SparkFun-Passives:PAD-JUMPER-3-2OF3_NC_BY_TRACE_YES_SILK_LARGE -> SparkFun-Passives:PAD-JUMPER-2-NC_BY_TRACE_YES_SILK
- U9: value MIC5205 -> PCA9306; device SparkFun-PowerIC:SOT23-5 -> SparkFun-DigitalIC:PCA9306DC-1:1
- moved R15 272.0 mm to (-103.0, -402.0)
- moved C13 226.0 mm to (-99.0, -430.0)
- moved C14 225.9 mm to (-93.0, -430.0)
- moved SJ4 222.2 mm to (-105.0, -426.0)
- moved JP2 220.1 mm to (-101.0, -417.0)
- moved U9 207.9 mm to (-104.0, -397.0)
- moved C12 187.3 mm to (-99.0, -395.0)
Connections:
- removed net 3.3V-REGULATED: C14.1, SJ4.3, U9.5
- removed net DCIN: Q1.2, U1.14
- removed net HV_SCL: JP2.1, R17.1, U8.6
- removed net HV_SDA: JP2.2, R16.1, U8.5
- removed net VOUT: C12.1, JP2.3, R16.2, R17.2, R18.2, SJ4.2
- removed net VSYS: C13.1, C6.1, C7.1, D1.A, D2.A, D3.A, L1.P$2, Q1.3, R13.2, R8.1, SJ4.1, U1.2, U1.4, U1.6, U9.1, U9.2
- new net GS1: BSS138_7.3, GIMBAL_SERVOS.S4, R43.2
- new net GS2: BSS138_1.3, GIMBAL_SERVOS.S3, R45.2
- new net GS3: BSS138_2.3, GIMBAL_SERVOS.S2, R47.2
- new net GS4: BSS138_3.3, GIMBAL_SERVOS.S1, R49.2
- new net I2C_1_SCL: R17.1, U8.6
- new net I2C_1_SDA: R16.1, U8.5
- new net I2C_2_SCL: R21.1, U9.6
- new net I2C_2_SDA: R15.1, U9.5
- new net MCU_RX: R29.2
- new net MCU_TX: R30.2
- new net N$26: C15.1, JP2.D-1, R25.1
- new net N$27: C16.1, JP2.D+1, R26.1
- new net N$28: R25.2, U11.12
- new net N$29: R26.2, U11.11
- new net N$30: SJ4.1, U11.17
- new net N$31: SJ5.1, U11.10
- new net N$32: R27.1, SJ4.2
- new net N$33: R28.1, SJ5.2
- new net N$34: D5.C, R27.2
- new net N$35: D6.C, R28.2
- new net N$36: R29.1, U11.20
- new net N$37: R30.1, U11.4
- new net POWER: POWER.P$C, U4.5
- new net VANT: U10.11
- new net VCC3.3: U10.3
- net 1.8V: now also BSS138_1.1, BSS138_2.1, BSS138_3.1, BSS138_7.1, C12.1, R23.2, R24.2, R44.1, R46.1, R48.1, R50.1, U9.1
- net 3.3V: now also C13.2, C6.1, C7.1, D3.A, L1.P$2, R13.2, R15.2, R16.2, R17.2, R18.2, R21.2, R22.2, R8.1, U1.14, U1.2, U1.4, U1.6, U11.14, U11.3; no longer U1.10, U1.8
- net 5V: now also C14.2, D1.A, D2.A, D5.A, D6.A, JP2.VBUS1, POWER.P$1, R31.2, R32.2, R33.2, R34.2, R35.2, R36.2, R37.2, R38.2, R39.2, R40.2, R41.2, R42.2, R43.1, R45.1, R47.1, R49.1, U11.15; no longer R15.2, U4.5
- net GND: now also C13.1, C14.1, C15.2, C16.2, JP2.GND1, JP2.SHIELD1, JP2.SHIELD2, JP2.SHIELD3, POWER.P$3, RESET.3, U10.23, U10.24, U10.25, U10.26, U10.27, U10.28, U10.29, U10.30, U10.6, U10.9, U11.16, U11.6, U9.4; no longer C13.2, C14.2, JP2.4, POWER.P$1, U9.3
- net GP12_PWM0: now also BSS138_7.2, R44.2; no longer GIMBAL_SERVOS.S4
- net GP13_PWM1: now also BSS138_1.2, R46.2; no longer GIMBAL_SERVOS.S3
- net GP182_PWM2: now also BSS138_2.2, R48.2; no longer GIMBAL_SERVOS.S2
- net GP183_PWM3: now also BSS138_3.2, R50.2; no longer GIMBAL_SERVOS.S1
- net GP27_I2C_6_SCL: now also R23.1, U9.2
- net GP28_I2C_6_SDA: now also R24.1, U9.3
- net M1: now also R31.1
- net M2: now also R32.1
- net M3: now also R33.1
- net M4: now also R34.1
- net M5: now also R35.1
- net M6: now also R36.1
- net MS1: now also R37.1
- net MS2: now also R38.1
- net MS3: now also R39.1
- net MS4: now also R40.1
- net MS5: now also R41.1
- net MS6: now also R42.1
- net N$15: now also RESET.1; no longer POWER.P$C
- net N$18: now also R22.1, U9.7, U9.8; no longer Q1.1, R15.1
