File: cudrone-board-mk-2.sch (EAGLE design)
At the start: 63 parts, among them Q1 200mA/50V, U1 EDISON_CONNECTOR_FULLMOUNTING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, U2 FTS31XS-U, U4 TPS62065, U5 USD-SOCKETNEW, U6 TXB0108, U8 PCA9306, U9 MIC5205

Commit message: Added logic level shifters to servos and changed how power input works
Parts:
- removed Q1: 200mA/50V, SparkFun-DiscreteSemi:MOSFET-NCHANNELBSS138
- added BSS138_1, BSS138_2, BSS138_3, BSS138_7: PMV22EN, eagle-library-edeca.net-v5:PMV22EN
- added C15, C16: 47pF, SparkFun-Capacitors:47PF-50V-5%(0603)
- added D5: RED, SparkFun-LED:LED-RED0603
- added D6: Yellow, SparkFun-LED:LED-YELLOW0603
- added R21: 10K, SparkFun-Resistors:10KOHM1/10W1%(0603)0603
- added R22: 200k, SparkFun-Resistors:200KOHM1/10W1%(0603)200K
- added R23, R24: DNP, SparkFun-Resistors:2.2KOHM1/10W1%(0603)
- added R25, R26: 27, SparkFun-Resistors:27OHM1/10W1%(0603)
- added R27, R28: 1K, SparkFun-Resistors:1KOHM1/10W1%(0603)
- added R29, R30: 100, SparkFun-Resistors:100OHM1/10W1%(0603)
- added R31, R32, R33, R34, R35, R36, R37, R38, R39, R40, R41, R42: (no value), SparkFun-Passives:RESISTOR0603-RES
- added R43, R44, R45, R46, R47, R48, R49, R50: 10k, SparkFun-Resistors:RESISTOR0805-RES
- added RESET: SWITCH-MOMENTARY-2PTH, SparkFun-Electromechanical:SWITCH-MOMENTARY-2PTH
- added SJ5: JUMPER-PAD-2-NC_BY_TRACE, SparkFun-Passives:JUMPER-PAD-2-NC_BY_TRACE
- added U10: A2235-H, A2235-H:A2235-H
- added U11: FTS31XS-U, SparkFun-DigitalIC:FT231XS
- C13, C14: value 10uF -> 0.1uF; device SparkFun-Capacitors:10UF-6.3V-20%(1206) -> SparkFun-Capacitors:0.1UF-25V(+80/-20%)(0603)
- JP2: value (none) -> USB_MICROB; device SparkFun-Connectors:M04SMD_RA_FEMALE -> SparkFun-Connectors:USB_MICROB_PLUGCONN-11752
- R14: value 120k -> 150k
- R15: value 1K -> 10K; device SparkFun-Resistors:1KOHM1/10W1%(0603) -> SparkFun-Resistors:10KOHM1/10W1%(0603)0603
- SJ4: value Power Select -> JUMPER-PAD-2-NC_BY_TRACE; device SparkFun-Passives:JUMPER-PAD-3-2OF3_NC_BY_TRACE_LARGE -> SparkFun-Passives:JUMPER-PAD-2-NC_BY_TRACE
- U9: value MIC5205 -> PCA9306; device SparkFun-PowerIC:MIC52053.3V -> SparkFun-DigitalIC:PCA9306PCA9306DC-1:1
Connections:
- removed net 3.3V-REGULATED: C14.1, SJ4.3, U9.OUT
- removed net DCIN: Q1.S, U1.DCIN
- removed net HV_SCL: JP2.1, R17.1, U8.SCL2
- removed net HV_SDA: JP2.2, R16.1, U8.SDA2
- removed net VOUT: C12.1, JP2.3, R16.2, R17.2, R18.2, SJ4.2
- removed net VSYS: C13.1, C6.1, C7.1, D1.A, D2.A, D3.A, L1.2, Q1.D, R13.2, R8.1, SJ4.1, U1.VSYS@1, U1.VSYS@2, U1.VSYS@3, U9.GND, U9.IN
- new net GS1: BSS138_7.D, GIMBAL_SERVOS.S4, R43.2
- new net GS2: BSS138_1.D, GIMBAL_SERVOS.S3, R45.2
- new net GS3: BSS138_2.D, GIMBAL_SERVOS.S2, R47.2
- new net GS4: BSS138_3.D, GIMBAL_SERVOS.S1, R49.2
- new net I2C_1_SCL: R17.1, U8.SCL2
- new net I2C_1_SDA: R16.1, U8.SDA2
- new net I2C_2_SCL: R21.1, U9.SCL2
- new net I2C_2_SDA: R15.1, U9.SDA2
- new net MCU_RX: R29.2
- new net MCU_TX: R30.2
- new net N$26: C15.1, JP2.D-, R25.1
- new net N$27: C16.1, JP2.D+, R26.1
- new net N$28: R25.2, U11.USBDM
- new net N$29: R26.2, U11.USBDP
- new net N$30: SJ4.1, U11.CBUS1
- new net N$31: SJ5.1, U11.CBUS2
- new net N$32: R27.1, SJ4.2
- new net N$33: R28.1, SJ5.2
- new net N$34: D5.C, R27.2
- new net N$35: D6.C, R28.2
- new net N$36: R29.1, U11.TXD
- new net N$37: R30.1, U11.RXD
- new net POWER: POWER.P, U4.EN
- net 1.8V: now also BSS138_1.G, BSS138_2.G, BSS138_3.G, BSS138_7.G, C12.1, R23.2, R24.2, R44.1, R46.1, R48.1, R50.1, U9.VREF1
- net 3.3V: now also C13.2, C6.1, C7.1, D3.A, L1.2, R13.2, R15.2, R16.2, R17.2, R18.2, R21.2, R22.2, R8.1, U1.DCIN, U1.VSYS@1, U1.VSYS@2, U1.VSYS@3, U11.!RESET, U11.VCCIO; no longer U1.3.3V@1, U1.3.3V@2
- net 5V: now also C14.2, D1.A, D2.A, D5.A, D6.A, JP2.VCC, POWER.O, R31.2, R32.2, R33.2, R34.2, R35.2, R36.2, R37.2, R38.2, R39.2, R40.2, R41.2, R42.2, R43.1, R45.1, R47.1, R49.1, U11.VCC; no longer R15.2, U4.EN
- net GND: now also C13.1, C14.1, C15.2, C16.2, JP2.GND, JP2.SHIELD, POWER.S, RESET.2, U11.GND@16, U11.GND@6, U9.GND; no longer C13.2, C14.2, JP2.4, POWER.O, U9.EN
- net GP12_PWM0: now also BSS138_7.S, R44.2; no longer GIMBAL_SERVOS.S4
- net GP13_PWM1: now also BSS138_1.S, R46.2; no longer GIMBAL_SERVOS.S3
- net GP182_PWM2: now also BSS138_2.S, R48.2; no longer GIMBAL_SERVOS.S2
- net GP183_PWM3: now also BSS138_3.S, R50.2; no longer GIMBAL_SERVOS.S1
- net GP27_I2C_6_SCL: now also R23.1, U9.SCL1
- net GP28_I2C_6_SDA: now also R24.1, U9.SDA1
- net M1: now also R31.1
- net M2: now also R32.1
- net M3: now also R33.1
- net M4: now also R34.1
- net M5: now also R35.1
- net M6: now also R36.1
- net MS1: now also R37.1
- net MS2: now also R38.1
- net MS3: now also R39.1
- net MS4: now also R40.1
- net MS5: now also R41.1
- net MS6: now also R42.1
- net N$15: now also RESET.1; no longer POWER.P
- net N$18: now also R22.1, U9.EN, U9.VREF2; no longer Q1.G, R15.1
Other:
- note added: "This sheet contains a usb port to connect to the edison's usb OTG port. It also contains a usb power regulator so that the usb port can be powered from usb. This power regulator is also connected to the usb uart bridge so that power to the board can be provided from both."
- note added: "This sheet contains the dspic that is used for reading the pwm signals from the radio reciver, and outputting the pwm signals to control the motor. They are i2c slaves to the main mcu. It also contains a usb connection for an enventual bootloader"
- note removed: "DCIN Enable Circuit Prevents Battery board from enabling DCIN"
- note removed: "Note: Default VOUT is 3.3v regulated."
- note removed: "This sheet contains a usb port to connect to the edison's usb OTG port. It also contains a usb power regulator so that the usb port can be powered from usb. This power regulator is also connected to the usb uart bridge so that power to the board can be provided from both. It also contains a hard wired port for the usb-webcam. It contains a switch to select between the two."
- note removed: "This sheet contains the dspic that is used for reading the pwm signals from the radio reciver, and outputting the pwm signals to control the motor. They are i2c slaves to the main mcu"
- moved on the sheet: C11, C12, C9, MOTOR_CONTROLLER, POWER, R16, R17, R18, R19, R20, U8

Commit message: Added flight sensors
Parts:
- added C17, C18: 0.1uF, SparkFun-Capacitors:CAP0603-CAP
- added C19: 120nF, SparkFun-Capacitors:CAP0603-CAP
- added C20: 6.8nF, SparkFun-Capacitors:CAP0603-CAP
- added DC1, DC15, DC16, DC2: 100nF, SparkFun-Capacitors:CAP0603-CAP
- added R51: 10k, SparkFun-Resistors:RESISTOR0805-RES
- added U$4: BMP280, BMP280:BMP280
- added U$5: BMP280PITOT, BMP280:BMP280PITOT
- added U12: BNO055, BNO055:BNO055
Connections:
- new net I2C0_SCL: U$4.SCL, U$5.SCL, U12.COM1
- new net I2C0_SDA: U$4.SDA, U$5.SDA, U12.COM0
- new net N$38: C18.1, U12.CAP
- new net NINT: U12.INT
- new net NRESET: R51.2, U12.NRESET
- net 3.3V: now also C17.1, C19.1, C20.1, DC1.1, DC15.1, DC16.1, DC2.1, R51.1, U$4.ADDRSEL, U$4.VCC, U$4.VDDIO, U$5.ADDRSEL, U$5.VCC, U$5.VDDIO, U12.NBOOT_LOAD_PIN, U12.VDD, U12.VDDIO
- net GND: now also C17.2, C18.2, C19.2, C20.2, DC1.2, DC15.2, DC16.2, DC2.2, U$4.GND, U$5.GND, U12.COM2, U12.COM3, U12.GND, U12.GNDIO, U12.PIN15, U12.PIN16, U12.PS0, U12.PS1
Other:
- note added: "Inside Temp/Pressure"
- note added: "Piot Tube"
- note added: "This sheet contains the flight sensors which are connected to the main mcu and needed to sustain flight. It contains the IMU, altimeter and the piot tube."
- note removed: "This sheet contains the flight sensors which are connected to the main mcu and needed to sustain flight. It contains the IMU, altimeter and the humidity sensor."
- moved on the sheet: C11, C12

Commit message: Added xbee and relavent connectors
Parts:
- added D30, D7, DC5, DC9: 10uF, SparkFun-Capacitors:CAP0603-CAP
- added DC13, DC4: 100nF, SparkFun-Capacitors:CAP0603-CAP
- added JP3, JP4: (no value), SparkFun-Connectors:M03PTH
- added U$6: XBEE, adafruit:XBEE
Connections:
- removed net UART_2_RX: U7.B2
- removed net UART_2_TX: U7.B1
- new net CON_RX: JP4.1, R7.2
- new net CON_TX: JP3.1, R6.2
- new net CTS_GPIO: U$6.CTS/DIO7
- new net RESET: U$6.RESET
- new net RTS_GPIO: U$6.RTS/AD6/DIO6
- new net XBEE_RX: U$6.DIN, U7.B1
- new net XBEE_RX_LOW: JP4.3, U7.A1
- new net XBEE_TX: U$6.DOUT, U7.B2
- new net XBEE_TX_LOW: JP3.3, U7.A2
- net 3.3V: now also D30.1, D7.1, DC13.1, DC4.1, DC5.1, DC9.1, U$6.VCC, U$6.VREF
- net GND: now also D30.2, D7.2, DC13.2, DC4.2, DC5.2, DC9.2, U$6.XBEE_GND
- net GP134_UART_2_RX: now also JP3.2; no longer R6.2, U7.A2
- net GP135_UART_2_TX: now also JP4.2; no longer R7.2, U7.A1

Commit message: Added GPS and relevent connections
Parts:
- added BSS138_4, BSS138_5, BSS138_6: PMV22EN, eagle-library-edeca.net-v5:PMV22EN
- added R52: 10k, SparkFun-Resistors:200KOHM1/10W1%(0603)200K
- added R53, R54: 2.2k, SparkFun-Resistors:2.2KOHM1/10W1%(0603)
- added R55, R56, R57, R58, R59, R60: 10k, SparkFun-Resistors:RESISTOR0805-RES
- R19, R20, R23, R24: value DNP -> 2.2k
Connections:
- new net GPS_NRST: BSS138_4.D, R55.2, U10.NRST
- new net GPS_ON_OFF: BSS138_5.D, R57.2, U10.ON_OFF
- new net GPS_WAKEUP: BSS138_6.D, R59.2, U10.WAKEUP
- new net N$39: R52.1, U10.GPIO6
- new net N$40: R52.2, U10.VOUT
- new net N$41: R53.1, U10.I2C_DIO
- new net N$42: R54.1, U10.I2C_CLK
- net 1.8V: now also BSS138_4.G, BSS138_5.G, BSS138_6.G, R56.1, R58.1, R60.1
- net 3.3V: now also R53.2, R54.2, R55.1, R57.1, R59.1, U10.VCC3.3
- net GND: now also U$6.GND, U10.GND@1, U10.GND@10, U10.GND@2, U10.GND@3, U10.GND@4, U10.GND@5, U10.GND@6, U10.GND@7, U10.GND@8, U10.GND@9; no longer U$6.XBEE_GND
- net GP165: now also BSS138_6.S, R60.2
- net GP44: now also BSS138_4.S, R56.2
- net GP45: now also BSS138_5.S, R58.2
- net UART_1_TX: now also U10.RXO, U10.TXO
Other:
- note added: "--------I2C--------"
- note added: "----SD_CARD----"
- note added: "---USB_OTG---"
- note added: "Console_UART"
- note added: "GPS_UART"
- note added: "Servos"

Commit message: Changed the dspic to a slightly different version so we can use it with simulink coder
Parts:
- removed MOTOR_CONTROLLER: DSPIC33EP512MC806-I/PT, DSPIC33EP512MC806:DSPIC33EP512MC806-I/PT
- added U13: DSPIC33EP512MU810-X_PF, DSPIC33EP512MU810-IPF:DSPIC33EP512MU810-X_PF
Other:
- moved on the sheet: D5, D6, R27, R28, SJ4, SJ5
Changed lines of the file:
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@@
 <part name="SUPPLY27" library="SparkFun-Aesthetics" deviceset="5V" device=""/>
 <part name="GND37" library="SparkFun-Aesthetics" deviceset="GND" device=""/>
-<part name="MOTOR_CONTROLLER" library="DSPIC33EP512MC806" deviceset="DSPIC33EP512MC806-I/PT" device=""/>
 <part name="GIMBAL_SERVOS1" library="Drone_Connectors" deviceset="3X4" device=""/>
 <part name="ESC" library="Drone_Connectors" deviceset="3X6" device=""/>
@@
 <part name="SUPPLY92" library="SparkFun-Aesthetics" deviceset="1.8V" device=""/>
 <part name="SUPPLY93" library="SparkFun-Aesthetics" deviceset="1.8V" device=""/>
+<part name="U13" library="DSPIC33EP512MU810-IPF" deviceset="DSPIC33EP512MU810-X_PF" device=""/>
 </parts>
 <sheets>
@@
 <instance part="FRAME6" gate="G$1" x="0" y="0"/>
 <instance part="FRAME6" gate="G$2" x="147.32" y="0"/>
-<instance part="MOTOR_CONTROLLER" gate="A" x="147.32" y="170.18"/>
 <instance part="JP2" gate="G$1" x="17.78" y="60.96" rot="MR0"/>
 <instance part="GND31" gate="1" x="27.94" y="45.72" rot="MR0"/>
@@
 <instance part="GND42" gate="1" x="43.18" y="45.72" rot="MR0"/>
 <instance part="SUPPLY46" gate="G$1" x="78.74" y="99.06"/>
-<instance part="SJ4" gate="G$1" x="134.62" y="55.88" smashed="yes" rot="R90">
-<attribute name="NAME" x="132.08" y="53.34" size="1.778" layer="95" rot="R90"/>
+<instance part="SJ4" gate="G$1" x="114.3" y="55.88" smashed="yes" rot="R90">
+<attribute name="NAME" x="111.76" y="53.34" size="1.778" layer="95" rot="R90"/>
 </instance>
-<instance part="SJ5" gate="G$1" x="142.24" y="55.88" smashed="yes" rot="R90">
-<attribute name="NAME" x="139.7" y="53.34" size="1.778" layer="95" rot="R90"/>
+<instance part="SJ5" gate="G$1" x="121.92" y="55.88" smashed="yes" rot="R90">
+<attribute name="NAME" x="119.38" y="53.34" size="1.778" layer="95" rot="R90"/>
 </instance>
-<instance part="R27" gate="G$1" x="134.62" y="68.58" rot="R90"/>
-<instance part="R28" gate="G$1" x="142.24" y="68.58" rot="R90"/>
-<instance part="D5" gate="G$1" x="134.62" y="78.74" rot="MR0"/>
-<instance part="D6" gate="G$1" x="142.24" y="78.74"/>
+<instance part="R27" gate="G$1" x="114.3" y="68.58" rot="R90"/>
+<instance part="R28" gate="G$1" x="121.92" y="68.58" rot="R90"/>
+<instance part="D5" gate="G$1" x="114.3" y="78.74" rot="MR0"/>
+<instance part="D6" gate="G$1" x="121.92" y="78.74"/>
 <instance part="R29" gate="G$1" x="93.98" y="73.66" smashed="yes">
 <attribute name="NAME" x="90.17" y="75.1586" size="1.778" layer="95"/>
@@
 <attribute name="VALUE" x="95.25" y="67.818" size="1.778" layer="96"/>
 </instance>
-<instance part="SUPPLY48" gate="G$1" x="134.62" y="83.82"/>
-<instance part="SUPPLY49" gate="G$1" x="142.24" y="83.82"/>
+<instance part="SUPPLY48" gate="G$1" x="114.3" y="83.82"/>
+<instance part="SUPPLY49" gate="G$1" x="121.92" y="83.82"/>
 <instance part="SUPPLY45" gate="G$1" x="68.58" y="99.06"/>
 <instance part="SUPPLY47" gate="G$1" x="45.72" y="76.2"/>
+<instance part="U13" gate="A" x="147.32" y="172.72"/>
 </instances>
 <busses>
@@
 <segment>
 <pinref part="D5" gate="G$1" pin="A"/>
-<wire x1="134.62" y1="81.28" x2="134.62" y2="83.82" width="0.1524" layer="91"/>
+<wire x1="114.3" y1="81.28" x2="114.3" y2="83.82" width="0.1524" layer="91"/>
 <pinref part="SUPPLY48" gate="G$1" pin="5V"/>
 </segment>
 <segment>
 <pinref part="D6" gate="G$1" pin="A"/>
-<wire x1="142.24" y1="81.28" x2="142.24" y2="83.82" width="0.1524" layer="91"/>
+<wire x1="121.92" y1="81.28" x2="121.92" y2="83.82" width="0.1524" layer="91"/>
 <pinref part="SUPPLY49" gate="G$1" pin="5V"/>
 </segment>
@@
 <pinref part="U11" gate="U$1" pin="CBUS1"/>
 <pinref part="SJ4" gate="G$1" pin="1"/>
-<wire x1="134.62" y1="50.8" x2="134.62" y2="48.26" width="0.1524" layer="91"/>
-<wire x1="134.62" y1="48.26" x2="86.36" y2="48.26" width="0.1524" layer="91"/>
+<wire x1="114.3" y1="50.8" x2="114.3" y2="48.26" width="0.1524" layer="91"/>
+<wire x1="114.3" y1="48.26" x2="86.36" y2="48.26" width="0.1524" layer="91"/>
 </segment>
 </net>
@@
 <pinref part="U11" gate="U$1" pin="CBUS2"/>
 <pinref part="SJ5" gate="G$1" pin="1"/>
-<wire x1="142.24" y1="50.8" x2="142.24" y2="45.72" width="0.1524" layer="91"/>
-<wire x1="142.24" y1="45.72" x2="86.36" y2="45.72" width="0.1524" layer="91"/>
+<wire x1="121.92" y1="50.8" x2="121.92" y2="45.72" width="0.1524" layer="91"/>
+<wire x1="121.92" y1="45.72" x2="86.36" y2="45.72" width="0.1524" layer="91"/>
 </segment>
 </net>
@@
 <pinref part="SJ4" gate="G$1" pin="2"/>
 <pinref part="R27" gate="G$1" pin="1"/>
-<wire x1="134.62" y1="63.5" x2="134.62" y2="60.96" width="0.1524" layer="91"/>
+<wire x1="114.3" y1="63.5" x2="114.3" y2="60.96" width="0.1524" layer="91"/>
 </segment>
 </net>
@@
 <pinref part="SJ5" gate="G$1" pin="2"/>
 <pinref part="R28" gate="G$1" pin="1"/>
-<wire x1="142.24" y1="63.5" x2="142.24" y2="60.96" width="0.1524" layer="91"/>
-</segment>
-</net>
+<wire x1="121.92" y1="63.5" x2="121.92" y2="60.96" width="0.1524" layer="91"/>
+</segment>
+</net>

Commit message: Fixed a few wiring issues and added some comments
Other:
- note added: "MCU is running at 3.3V so pullups to make output signal at 5V and the mcu is pulling down."
- note added: "This rather strange looking connection allows for the usb to be powered from either direction."
Changed lines of the file:
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@@
 <?xml version="1.0" encoding="utf-8"?>
 <!DOCTYPE eagle SYSTEM "eagle.dtd">
-<eagle version="8.0.0">
+<eagle version="8.2.2">
 <drawing>
 <settings>
@@
 <text x="172.72" y="144.78" size="1.778" layer="97" rot="R270">----SD_CARD----</text>
 <text x="170.18" y="66.04" size="1.778" layer="97" rot="R270">--------I2C--------</text>
-<text x="167.64" y="68.58" size="1.778" layer="97" rot="R90">GPS_UART</text>
+<text x="175.26" y="111.76" size="1.778" layer="97" rot="R90">GPS_UART</text>
 </plain>
 <instances>
@@
 is also connected to the usb uart bridge so that power to
 the board can be provided from both. </text>
+<text x="43.18" y="162.56" size="1.778" layer="91">This rather strange looking
+connection allows for the
+usb to be powered from
+either direction.</text>
 </plain>
 <instances>
@@
  and landing gear, the connections to the reciver
 and the connections to the esc</text>
+<text x="137.16" y="78.74" size="1.778" layer="91">MCU is running at 3.3V so pullups to make output signal at 5V and the mcu is pulling down.</text>
 </plain>
 <instances>
